Commit message: Add baseline 4 dof

File: src/my_robot_arm/urdf/arm.urdf.xacro (robot description, xacro)
@@ -1,70 +1,205 @@
 <?xml version="1.0"?>
-<robot name="2dof_arm" xmlns:xacro="http://www.ros.org/wiki/xacro">
-  <!-- Base Link -->
-  <link name="base_link">
-    <inertial>
-      <mass value="1.0"/>
-      <origin xyz="0 0 0" rpy="0 0 0"/>
-      <inertia ixx="0.01" iyy="0.01" izz="0.01" ixy="0" ixz="0" iyz="0"/>
-    </inertial>
-    <visual>
-      <geometry><cylinder length="0.1" radius="0.05"/></geometry>
-      <material name="base_material">
-        <color rgba="0.3 0.3 0.3 1"/>
-      </material>
-    </visual>
-    <collision>
-      <geometry><cylinder length="0.1" radius="0.05"/></geometry>
-    </collision>
-  </link>
-  <!-- Joint 1 -->
-  <joint name="joint1" type="revolute">
-    <parent link="base_link"/>
-    <child link="link1"/>
-    <origin xyz="0 0 0.05" rpy="0 0 0"/>
-    <axis xyz="0 0 1"/>
-    <limit effort="10.0" velocity="1.0" lower="-1.57" upper="1.57"/>
-  </joint>
-  <!-- Link 1 -->
-  <link name="link1">
-    <inertial>
-      <mass value="0.8"/>
-      <origin xyz="0 0 0" rpy="0 0 0"/>
-      <inertia ixx="0.005" iyy="0.005" izz="0.005" ixy="0" ixz="0" iyz="0"/>
-    </inertial>
-    <visual>
-      <geometry><box size="0.3 0.05 0.05"/></geometry>
-      <material name="link1_material">
-        <color rgba="0.6 0.2 0.2 1"/>
-      </material>
-    </visual>
-    <collision>
-      <geometry><box size="0.3 0.05 0.05"/></geometry>
-    </collision>
-  </link>
-  <!-- Joint 2 -->
-  <joint name="joint2" type="revolute">
-    <parent link="link1"/>
-    <child link="link2"/>
-    <origin xyz="0.15 0 0" rpy="0 0 0"/>
-    <axis xyz="0 0 1"/>
-    <limit effort="10.0" velocity="1.0" lower="-1.57" upper="1.57"/>
-  </joint>
-  <!-- Link 2 -->
-  <link name="link2">
-    <inertial>
-      <mass value="0.5"/>
-      <origin xyz="0 0 0" rpy="0 0 0"/>
-      <inertia ixx="0.003" iyy="0.003" izz="0.003" ixy="0" ixz="0" iyz="0"/>
-    </inertial>
-    <visual>
-      <geometry><box size="0.3 0.05 0.05"/></geometry>
-      <material name="link2_material">
-        <color rgba="0.2 0.2 0.6 1"/>
-      </material>
-    </visual>
-    <collision>
-      <geometry><box size="0.3 0.05 0.05"/></geometry>
-    </collision>
-  </link>
+<robot name="4dof_arm" xmlns:xacro="http://www.ros.org/wiki/xacro">
+    <!-- World link -->
+    <link name="world"/>
+    <!-- Base Link -->
+    <link name="base_link">
+        <inertial>
+            <mass value="1.0"/>
+            <origin rpy="0 0 0" xyz="0 0 0.025"/>
+            <inertia ixx="0.0027" iyy="0.0027" izz="0.005" ixy="0" ixz="0" iyz="0"/>
+        </inertial>
+        <visual>
+            <geometry>
+                <cylinder length="0.05" radius="0.1"/>
+            </geometry>
+            <material name="silver">
+                <color rgba="0.75 0.75 0.75 1"/>
+            </material>
+            <origin rpy="0 0 0" xyz="0 0 0.025"/>
+        </visual>
+        <collision>
+            <geometry>
+                <cylinder length="0.05" radius="0.1"/>
+            </geometry>
+            <origin rpy="0 0 0" xyz="0 0 0.025"/>
+        </collision>
+    </link>
+    <!-- Fixed joint connecting world to base_link -->
+    <joint name="fixed" type="fixed">
+        <parent link="world"/>
+        <child link="base_link"/>
+    </joint>
+    <!-- Link 1 (First vertical link) -->
+    <link name="link1">
+        <inertial>
+            <mass value="1.0"/>
+            <origin rpy="0 0 0" xyz="0 0 0.15"/>
+            <inertia ixx="0.01396" iyy="0.01396" izz="0.00125" ixy="0" ixz="0" iyz="0"/>
+        </inertial>
+        <visual>
+            <geometry>
+                <cylinder length="0.3" radius="0.04"/>
+            </geometry>
+            <material name="orange">
+                <color rgba="1.0 0.6 0.0 1"/>
+            </material>
+            <origin rpy="0 0 0" xyz="0 0 0.15"/>
+        </visual>
+        <collision>
+            <geometry>
+                <cylinder length="0.3" radius="0.04"/>
+            </geometry>
+            <origin rpy="0 0 0" xyz="0 0 0.15"/>
+        </collision>
+    </link>
+    <!-- Joint 1 (Rotates around Z axis) -->
+    <joint name="joint1" type="continuous">
+        <axis xyz="0 0 1"/>
+        <parent link="base_link"/>
+        <child link="link1"/>
+        <origin rpy="0 0 0" xyz="0 0 0.05"/>
+    </joint>
+    <!-- Link 2 (Upper arm) -->
+    <link name="link2">
+        <inertial>
+            <mass value="0.8"/>
+            <origin rpy="0 0 0" xyz="0 0 0.15"/>
+            <inertia ixx="0.0078" iyy="0.0078" izz="0.0010" ixy="0" ixz="0" iyz="0"/>
+        </inertial>
+        <visual>
+            <geometry>
+                <cylinder length="0.3" radius="0.04"/>
+            </geometry>
+            <material name="orange">
+                <color rgba="1.0 0.6 0.0 1"/>
+            </material>
+            <origin rpy="0 0 0" xyz="0 0 0.15"/>
+        </visual>
+        <collision>
+            <geometry>
+                <cylinder length="0.3" radius="0.04"/>
+            </geometry>
+            <origin rpy="0 0 0" xyz="0 0 0.15"/>
+        </collision>
+    </link>
+    <!-- Joint 2 (Shoulder - rotates around Y axis) -->
+    <joint name="joint2" type="revolute">
+        <axis xyz="0 1 0"/>
+        <limit velocity="1.0" effort="30.0" upper="1.5708" lower="-1.5708"/>
+        <parent link="link1"/>
+        <child link="link2"/>
+        <origin rpy="0 1.5708 0" xyz="0 0 0.3"/>
+    </joint>
+    <!-- Link 3 (Lower arm) -->
+    <link name="link3">
+        <inertial>
+            <mass value="0.6"/>
+            <origin rpy="0 0 0" xyz="0 0 0.125"/>
+            <inertia ixx="0.0045" iyy="0.0045" izz="0.0008" ixy="0" ixz="0" iyz="0"/>
+        </inertial>
+        <visual>
+            <geometry>
+                <cylinder length="0.25" radius="0.035"/>
+            </geometry>
+            <material name="orange">
+                <color rgba="1.0 0.6 0.0 1"/>
+            </material>
+            <origin rpy="0 0 0" xyz="0 0 0.125"/>
+        </visual>
+        <collision>
+            <geometry>
+                <cylinder length="0.25" radius="0.035"/>
+            </geometry>
+            <origin rpy="0 0 0" xyz="0 0 0.125"/>
+        </collision>
+    </link>
+    <!-- Joint 3 (Elbow - rotates around Y axis) -->
+    <joint name="joint3" type="revolute">
+        <axis xyz="0 1 0"/>
+        <limit velocity="1.0" effort="30.0" upper="1.5708" lower="-1.5708"/>
+        <parent link="link2"/>
+        <child link="link3"/>
+        <origin rpy="0 0 0" xyz="0 0 0.3"/>
+    </joint>
+    <!-- Link 4 (End effector) -->
+    <link name="end_effector">
+        <inertial>
+            <mass value="0.4"/>
+            <origin rpy="0 0 0" xyz="0 0 0.1"/>
+            <inertia ixx="0.0030" iyy="0.0030" izz="0.0006" ixy="0" ixz="0" iyz="0"/>
+        </inertial>
+        <visual>
+            <geometry>
+                <cylinder length="0.2" radius="0.03"/>
+            </geometry>
+            <material name="orange">
+                <color rgba="1.0 0.6 0.0 1"/>
+            </material>
+            <origin rpy="0 0 0" xyz="0 0 0.1"/>
+        </visual>
+        <collision>
+            <geometry>
+                <cylinder length="0.2" radius="0.03"/>
+            </geometry>
+            <origin rpy="0 0 0" xyz="0 0 0.1"/>
+        </collision>
+    </link>
+    <!-- Joint 4 (Wrist - rotates around Z axis) -->
+    <joint name="joint4" type="continuous">
+        <axis xyz="0 0 1"/>
+        <parent link="link3"/>
+        <child link="end_effector"/>
+        <origin rpy="0 0 0" xyz="0 0 0.25"/>
+    </joint>
+    <!-- Transmissions for ROS control -->
+    <transmission name="tran1">
+        <type>transmission_interface/SimpleTransmission</type>
+        <joint name="joint1">
+            <hardwareInterface>hardware_interface/PositionJointInterface</hardwareInterface>
+        </joint>
+        <actuator name="motor1">
+            <hardwareInterface>hardware_interface/PositionJointInterface</hardwareInterface>
+            <mechanicalReduction>1</mechanicalReduction>
+        </actuator>
+    </transmission>
+    <transmission name="tran2">
+        <type>transmission_interface/SimpleTransmission</type>
+        <joint name="joint2">
+            <hardwareInterface>hardware_interface/PositionJointInterface</hardwareInterface>
+        </joint>
+        <actuator name="motor2">
+            <hardwareInterface>hardware_interface/PositionJointInterface</hardwareInterface>
+            <mechanicalReduction>1</mechanicalReduction>
+        </actuator>
+    </transmission>
+    <transmission name="tran3">
+        <type>transmission_interface/SimpleTransmission</type>
+        <joint name="joint3">
+            <hardwareInterface>hardware_interface/PositionJointInterface</hardwareInterface>
+        </joint>
+        <actuator name="motor3">
+            <hardwareInterface>hardware_interface/PositionJointInterface</hardwareInterface>
+            <mechanicalReduction>1</mechanicalReduction>
+        </actuator>
+    </transmission>
+    <transmission name="tran4">
+        <type>transmission_interface/SimpleTransmission</type>
+        <joint name="joint4">
+            <hardwareInterface>hardware_interface/PositionJointInterface</hardwareInterface>
+        </joint>
+        <actuator name="motor4">
+            <hardwareInterface>hardware_interface/PositionJointInterface</hardwareInterface>
+            <mechanicalReduction>1</mechanicalReduction>
+        </actuator>
+    </transmission>
+    <!-- Gazebo plugins for ROS2 control -->
+    <gazebo>
+        <plugin name="control" filename="libgazebo_ros_control.so"/>
+    </gazebo>
+    <gazebo>
+        <plugin name="joint_state_publisher" filename="libgazebo_ros_joint_state_publisher.so">
+            <jointName>joint1, joint2, joint3, joint4</jointName>
+        </plugin>
+    </gazebo>
 </robot>

Commit message: Add another urdf more beautiful

File: src/my_robot_arm/urdf/arm.urdf.xacro (robot description, xacro)
@@ -1,205 +1,294 @@
-<?xml version="1.0"?>
-<robot name="4dof_arm" xmlns:xacro="http://www.ros.org/wiki/xacro">
-    <!-- World link -->
-    <link name="world"/>
-    <!-- Base Link -->
-    <link name="base_link">
-        <inertial>
-            <mass value="1.0"/>
-            <origin rpy="0 0 0" xyz="0 0 0.025"/>
-            <inertia ixx="0.0027" iyy="0.0027" izz="0.005" ixy="0" ixz="0" iyz="0"/>
-        </inertial>
-        <visual>
-            <geometry>
-                <cylinder length="0.05" radius="0.1"/>
-            </geometry>
-            <material name="silver">
-                <color rgba="0.75 0.75 0.75 1"/>
-            </material>
-            <origin rpy="0 0 0" xyz="0 0 0.025"/>
-        </visual>
-        <collision>
-            <geometry>
-                <cylinder length="0.05" radius="0.1"/>
-            </geometry>
-            <origin rpy="0 0 0" xyz="0 0 0.025"/>
-        </collision>
-    </link>
-    <!-- Fixed joint connecting world to base_link -->
-    <joint name="fixed" type="fixed">
-        <parent link="world"/>
-        <child link="base_link"/>
-    </joint>
-    <!-- Link 1 (First vertical link) -->
-    <link name="link1">
-        <inertial>
-            <mass value="1.0"/>
-            <origin rpy="0 0 0" xyz="0 0 0.15"/>
-            <inertia ixx="0.01396" iyy="0.01396" izz="0.00125" ixy="0" ixz="0" iyz="0"/>
-        </inertial>
-        <visual>
-            <geometry>
-                <cylinder length="0.3" radius="0.04"/>
-            </geometry>
-            <material name="orange">
-                <color rgba="1.0 0.6 0.0 1"/>
-            </material>
-            <origin rpy="0 0 0" xyz="0 0 0.15"/>
-        </visual>
-        <collision>
-            <geometry>
-                <cylinder length="0.3" radius="0.04"/>
-            </geometry>
-            <origin rpy="0 0 0" xyz="0 0 0.15"/>
-        </collision>
-    </link>
-    <!-- Joint 1 (Rotates around Z axis) -->
-    <joint name="joint1" type="continuous">
-        <axis xyz="0 0 1"/>
-        <parent link="base_link"/>
-        <child link="link1"/>
-        <origin rpy="0 0 0" xyz="0 0 0.05"/>
-    </joint>
-    <!-- Link 2 (Upper arm) -->
-    <link name="link2">
-        <inertial>
-            <mass value="0.8"/>
-            <origin rpy="0 0 0" xyz="0 0 0.15"/>
-            <inertia ixx="0.0078" iyy="0.0078" izz="0.0010" ixy="0" ixz="0" iyz="0"/>
-        </inertial>
-        <visual>
-            <geometry>
-                <cylinder length="0.3" radius="0.04"/>
-            </geometry>
-            <material name="orange">
-                <color rgba="1.0 0.6 0.0 1"/>
-            </material>
-            <origin rpy="0 0 0" xyz="0 0 0.15"/>
-        </visual>
-        <collision>
-            <geometry>
-                <cylinder length="0.3" radius="0.04"/>
-            </geometry>
-            <origin rpy="0 0 0" xyz="0 0 0.15"/>
-        </collision>
-    </link>
-    <!-- Joint 2 (Shoulder - rotates around Y axis) -->
-    <joint name="joint2" type="revolute">
-        <axis xyz="0 1 0"/>
-        <limit velocity="1.0" effort="30.0" upper="1.5708" lower="-1.5708"/>
-        <parent link="link1"/>
-        <child link="link2"/>
-        <origin rpy="0 1.5708 0" xyz="0 0 0.3"/>
-    </joint>
-    <!-- Link 3 (Lower arm) -->
-    <link name="link3">
-        <inertial>
-            <mass value="0.6"/>
-            <origin rpy="0 0 0" xyz="0 0 0.125"/>
-            <inertia ixx="0.0045" iyy="0.0045" izz="0.0008" ixy="0" ixz="0" iyz="0"/>
-        </inertial>
-        <visual>
-            <geometry>
-                <cylinder length="0.25" radius="0.035"/>
-            </geometry>
-            <material name="orange">
-                <color rgba="1.0 0.6 0.0 1"/>
-            </material>
-            <origin rpy="0 0 0" xyz="0 0 0.125"/>
-        </visual>
-        <collision>
-            <geometry>
-                <cylinder length="0.25" radius="0.035"/>
-            </geometry>
-            <origin rpy="0 0 0" xyz="0 0 0.125"/>
-        </collision>
-    </link>
-    <!-- Joint 3 (Elbow - rotates around Y axis) -->
-    <joint name="joint3" type="revolute">
-        <axis xyz="0 1 0"/>
-        <limit velocity="1.0" effort="30.0" upper="1.5708" lower="-1.5708"/>
-        <parent link="link2"/>
-        <child link="link3"/>
-        <origin rpy="0 0 0" xyz="0 0 0.3"/>
-    </joint>
-    <!-- Link 4 (End effector) -->
-    <link name="end_effector">
-        <inertial>
-            <mass value="0.4"/>
-            <origin rpy="0 0 0" xyz="0 0 0.1"/>
-            <inertia ixx="0.0030" iyy="0.0030" izz="0.0006" ixy="0" ixz="0" iyz="0"/>
-        </inertial>
-        <visual>
-            <geometry>
-                <cylinder length="0.2" radius="0.03"/>
-            </geometry>
-            <material name="orange">
-                <color rgba="1.0 0.6 0.0 1"/>
-            </material>
-            <origin rpy="0 0 0" xyz="0 0 0.1"/>
-        </visual>
-        <collision>
-            <geometry>
-                <cylinder length="0.2" radius="0.03"/>
-            </geometry>
-            <origin rpy="0 0 0" xyz="0 0 0.1"/>
-        </collision>
-    </link>
-    <!-- Joint 4 (Wrist - rotates around Z axis) -->
-    <joint name="joint4" type="continuous">
-        <axis xyz="0 0 1"/>
-        <parent link="link3"/>
-        <child link="end_effector"/>
-        <origin rpy="0 0 0" xyz="0 0 0.25"/>
-    </joint>
-    <!-- Transmissions for ROS control -->
-    <transmission name="tran1">
-        <type>transmission_interface/SimpleTransmission</type>
-        <joint name="joint1">
-            <hardwareInterface>hardware_interface/PositionJointInterface</hardwareInterface>
-        </joint>
-        <actuator name="motor1">
-            <hardwareInterface>hardware_interface/PositionJointInterface</hardwareInterface>
-            <mechanicalReduction>1</mechanicalReduction>
-        </actuator>
-    </transmission>
-    <transmission name="tran2">
-        <type>transmission_interface/SimpleTransmission</type>
-        <joint name="joint2">
-            <hardwareInterface>hardware_interface/PositionJointInterface</hardwareInterface>
-        </joint>
-        <actuator name="motor2">
-            <hardwareInterface>hardware_interface/PositionJointInterface</hardwareInterface>
-            <mechanicalReduction>1</mechanicalReduction>
-        </actuator>
-    </transmission>
-    <transmission name="tran3">
-        <type>transmission_interface/SimpleTransmission</type>
-        <joint name="joint3">
-            <hardwareInterface>hardware_interface/PositionJointInterface</hardwareInterface>
-        </joint>
-        <actuator name="motor3">
-            <hardwareInterface>hardware_interface/PositionJointInterface</hardwareInterface>
-            <mechanicalReduction>1</mechanicalReduction>
-        </actuator>
-    </transmission>
-    <transmission name="tran4">
-        <type>transmission_interface/SimpleTransmission</type>
-        <joint name="joint4">
-            <hardwareInterface>hardware_interface/PositionJointInterface</hardwareInterface>
-        </joint>
-        <actuator name="motor4">
-            <hardwareInterface>hardware_interface/PositionJointInterface</hardwareInterface>
-            <mechanicalReduction>1</mechanicalReduction>
-        </actuator>
-    </transmission>
-    <!-- Gazebo plugins for ROS2 control -->
-    <gazebo>
-        <plugin name="control" filename="libgazebo_ros_control.so"/>
-    </gazebo>
-    <gazebo>
-        <plugin name="joint_state_publisher" filename="libgazebo_ros_joint_state_publisher.so">
-            <jointName>joint1, joint2, joint3, joint4</jointName>
-        </plugin>
-    </gazebo>
+<robot name="arm">
+	<link name="world"/>
+	<link name="base_link">
+		<inertial>
+			<mass value="1.0"/>
+			<origin rpy="0 0 0" xyz="0 0 0.025"/>
+			<inertia ixx="0.0027" iyy="0.0027" izz="0.005" ixy="0" ixz="0" iyz="0"/>
+		</inertial>
+		<visual>
+			<geometry>
+				<cylinder length="0.05" radius="0.1"/>
+			</geometry>
+			<material name="silver">
+				<color rgba="0.75 0.75 0.75 1"/>
+			</material>
+			<origin rpy="0 0 0" xyz="0 0 0.025"/>
+		</visual>
+		<collision>
+			<geometry>
+				<cylinder length="0.05" radius="0.1"/>
+			</geometry>
+			<origin rpy="0 0 0" xyz="0 0 0.025"/>
+		</collision>
+	</link>
+	<joint name="fixed" type="fixed">
+		<parent link="world"/>
+		<child link="base_link"/>
+	</joint>
+	<link name="torso">
+		<inertial>
+			<mass value="1.0"/>
+			<origin rpy="0 0 0" xyz="0 0 0.25"/>
+			<inertia ixx="0.02146" iyy="0.02146" izz="0.00125" ixy="0" ixz="0" iyz="0"/>
+		</inertial>
+		<visual>
+			<geometry>
+				<cylinder length="0.5" radius="0.05"/>
+			</geometry>
+			<material name="silver">
+				<color rgba="0.75 0.75 0.75 1"/>
+			</material>
+			<origin rpy="0 0 0" xyz="0.0 0.0 0.25"/>
+		</visual>
+		<collision>
+			<geometry>
+				<cylinder length="0.5" radius="0.05"/>
+			</geometry>
+			<origin rpy="0 0 0" xyz="0.0 0.0 0.25"/>
+		</collision>
+	</link>
+	<joint name="hip" type="continuous">
+		<axis xyz="0 0 1"/>
+		<parent link="base_link"/>
+		<child link="torso"/>
+		<origin rpy="0 0 0" xyz="0 0 0.05"/>
+	</joint>
+	<link name="upper_arm">
+		<inertial>
+			<mass value="1.0"/>
+			<origin rpy="0 0 0" xyz="0 0 0.2"/>
+			<inertia ixx="0.01396" iyy="0.01396" izz="0.00125" ixy="0" ixz="0" iyz="0"/>
+		</inertial>
+		<visual>
+			<geometry>
+				<cylinder length="0.4" radius="0.05"/>
+			</geometry>
+			<material name="silver"/>
+			<origin rpy="0 0 0" xyz="0 0 0.2"/>
+		</visual>
+		<collision>
+			<geometry>
+				<cylinder length="0.4" radius="0.05"/>
+			</geometry>
+			<origin rpy="0 0 0" xyz="0 0 0.2"/>
+		</collision>
+	</link>
+	<joint name="shoulder" type="revolute">
+		<axis xyz="0 1 0"/>
+		<limit velocity="1.0" effort="30.0" upper="0.6981" lower="-1.5708"/>
+		<parent link="torso"/>
+		<child link="upper_arm"/>
+		<origin rpy="0 1.5708 0" xyz="0.0 -0.1 0.45"/>
+	</joint>
+	<link name="lower_arm">
+		<inertial>
+			<mass value="1.0"/>
+			<origin rpy="0 0 0" xyz="0 0 0.2"/>
+			<inertia ixx="0.01396" iyy="0.01396" izz="0.00125" ixy="0" ixz="0" iyz="0"/>
+		</inertial>
+		<visual>
+			<geometry>
+				<cylinder length="0.4" radius="0.05"/>
+			</geometry>
+			<material name="silver"/>
+			<origin rpy="0 0 0" xyz="0 0 0.2"/>
+		</visual>
+		<collision>
+			<geometry>
+				<cylinder length="0.4" radius="0.05"/>
+			</geometry>
+			<origin rpy="0 0 0" xyz="0 0 0.2"/>
+		</collision>
+	</link>
+	<joint name="elbow" type="revolute">
+		<axis xyz="0 1 0"/>
+		<limit velocity="1.0" effort="30.0" upper="1.5708" lower="-1.5708"/>
+		<parent link="upper_arm"/>
+		<child link="lower_arm"/>
+		<origin rpy="0 0 0" xyz="0.0 0.1 0.35"/>
+	</joint>
+	<link name="hand">
+		<inertial>
+			<mass value="1.0"/>
+			<inertia ixx="0.00042" iyy="0.00042" izz="0.00042" ixy="0" ixz="0" iyz="0"/>
+		</inertial>
+		<visual>
+			<geometry>
+				<box size="0.05 0.05 0.05"/>
+			</geometry>
+			<material name="silver"/>
+		</visual>
+		<collision>
+			<geometry>
+				<box size="0.05 0.05 0.05"/>
+			</geometry>
+		</collision>
+	</link>
+	<joint name="wrist" type="continuous">
+		<axis xyz="0 1 0"/>
+		<parent link="lower_arm"/>
+		<child link="hand"/>
+		<origin rpy="0 0 0" xyz="0.0 0.0 0.425"/>
+	</joint>
+	<link name="left_gripper_base">
+		<inertial>
+			<mass value="0.01"/>
+			<inertia ixx="8.23e-8" iyy="8.23e-8" izz="3.47e-7" ixy="0" ixz="0" iyz="0"/>
+		</inertial>
+		<visual>
+			<geometry>
+				<box size="0.005 0.005 0.02"/>
+			</geometry>
+			<material name="silver"/>
+		</visual>
+		<collision>
+			<geometry>
+				<box size="0.005 0.005 0.02"/>
+			</geometry>
+		</collision>
+	</link>
+	<joint name="l_g_base" type="revolute">
+		<axis xyz="1 0 0"/>
+		<limit velocity="1.0" effort="30.0" lower="0" upper="0.5236"/>
+		<origin rpy="-0.9162 0 0" xyz="0 0.02 0.035"/>
+		<parent link="hand"/>
+		<child link="left_gripper_base"/>
+	</joint>
+	<link name="right_gripper_base">
+		<inertial>
+			<mass value="0.01"/>
+			<inertia ixx="8.23e-8" iyy="8.23e-8" izz="3.47e-7" ixy="0" ixz="0" iyz="0"/>
+		</inertial>
+		<visual>
+			<geometry>
+				<box size="0.005 0.005 0.02"/>
+			</geometry>
+			<material name="silver"/>
+		</visual>
+		<collision>
+			<geometry>
+				<box size="0.005 0.005 0.02"/>
+			</geometry>
+		</collision>
+	</link>
+	<joint name="r_g_base" type="revolute">
+		<axis xyz="1 0 0"/>
+		<limit velocity="1.0" effort="100.0" upper="0" lower="-0.5236"/>
+		<origin rpy="0.9162 0 0" xyz="0 -0.02 0.035"/>
+		<parent link="hand"/>
+		<child link="right_gripper_base"/>
+	</joint>
+	<link name="left_gripper_finger">
+		<inertial>
+			<mass value="0.01"/>
+			<inertia ixx="1.57e-7" iyy="1.57e-7" izz="6.8e-7" ixy="0" ixz="0" iyz="0"/>
+		</inertial>
+		<visual>
+			<geometry>
+				<box size="0.008 0.008 0.05"/>
+			</geometry>
+			<material name="silver"/>
+		</visual>
+		<collision>
+			<geometry>
+				<box size="0.008 0.008 0.05"/>
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